Commit message: feat(moveit): add sim_mode argument and real-robot launch
Parametrizes the MoveIt config to support three hardware backends
selectable at launch time without rebuilding:

- mock   (default): mock_components/GenericSystem (RViz testing)
- gazebo: gz_ros2_control/GazeboSimSystem (uses abb_irb14050_gazebo)
- real:   placeholder for EGM hardware interface; in practice the
          real-robot path uses the egm_moveit_executor action server
          instead of a ros2_control plugin (see moveit_real.launch.py)

Changes:

- abb_irb14050.ros2_control.xacro: wraps the plugin in xacro:if blocks
  keyed on ${sim_mode}, with a 'real' branch left as a comment for
  future EGM hardware_interface integration.
- abb_irb14050.urdf.xacro: declares the sim_mode argument, forwards it
  to the ros2_control macro, and conditionally injects the
  <gazebo><plugin gz_ros2_control/></gazebo> block when
  sim_mode == 'gazebo'.
- joint_limits.yaml: max_velocity reduced from ~pi rad/s (and
  ~6.98 rad/s for joints 5-7) to a uniform 0.5 rad/s. Tuned for safe
  real-robot operation; the team can raise these for faster mock-mode
  validation. Adds goal_position_tolerance and goal_velocity_tolerance
  per joint.
- moveit_controllers.yaml: adds trajectory_execution block with
  generous tolerances (allowed_execution_duration_scaling: 5.0,
  allowed_goal_duration_margin: 5.0, allowed_start_tolerance: 0.05)
  so MoveIt does not abort trajectories due to the EGM bridge slew
  rate cap.
- launch/moveit_real.launch.py: NEW. Brings up move_group + RViz +
  egm_bridge + egm_moveit_executor. Does not start ros2_control_node
  or mock controllers — the executor takes the controller's place
  in this mode.

README updated with the three modes, build/use instructions per mode,
and notes on the joint_limits trade-off and the trajectory_execution
tolerances.

File: irb14050_ws/src/abb_irb14050_moveit_config/config/abb_irb14050.ros2_control.xacro (robot description, xacro)
@@ -1,10 +1,25 @@
 <?xml version="1.0"?>
 <robot xmlns:xacro="http://www.ros.org/wiki/xacro">
-    <xacro:macro name="abb_irb14050_ros2_control" params="name initial_positions_file">
+    <!--
+        sim_mode: selects the hardware interface plugin loaded by ros2_control.
+            - "mock"   : mock_components/GenericSystem  (no physics, RViz testing)
+            - "gazebo" : gz_ros2_control/GazeboSimSystem (Gazebo Harmonic)
+            - "real"   : (placeholder — wire EGM hardware interface here in the future)
+    -->
+    <xacro:macro name="abb_irb14050_ros2_control" params="name initial_positions_file sim_mode:=mock">
         <xacro:property name="initial_positions" value="${xacro.load_yaml(initial_positions_file)['initial_positions']}"/>
         <ros2_control name="${name}" type="system">
             <hardware>
-                <!-- By default, set up controllers for simulation. This won't work on real hardware -->
-                <plugin>mock_components/GenericSystem</plugin>
+                <xacro:if value="${sim_mode == 'mock'}">
+                    <plugin>mock_components/GenericSystem</plugin>
+                </xacro:if>
+                <xacro:if value="${sim_mode == 'gazebo'}">
+                    <plugin>gz_ros2_control/GazeboSimSystem</plugin>
+                </xacro:if>
+                <!-- Future: real robot via EGM
+                <xacro:if value="${sim_mode == 'real'}">
+                    <plugin>abb_irb14050_egm/EGMHardwareInterface</plugin>
+                </xacro:if>
+                -->
             </hardware>
             <joint name="joint_1">

File: irb14050_ws/src/abb_irb14050_moveit_config/config/abb_irb14050.urdf.xacro (robot description, xacro)
@@ -2,8 +2,20 @@
 <robot xmlns:xacro="http://www.ros.org/wiki/xacro" name="abb_irb14050">
     <xacro:arg name="initial_positions_file" default="initial_positions.yaml" />
+    <xacro:arg name="sim_mode" default="mock" />
     <!-- Import abb_irb14050 urdf file -->
     <xacro:include filename="$(find abb_irb14050_description)/urdf/abb_irb14050.urdf" />
     <!-- Import control_xacro -->
     <xacro:include filename="abb_irb14050.ros2_control.xacro" />
-    <xacro:abb_irb14050_ros2_control name="FakeSystem" initial_positions_file="$(arg initial_positions_file)"/>
+    <xacro:abb_irb14050_ros2_control
+        name="ABB_IRB14050_System"
+        initial_positions_file="$(arg initial_positions_file)"
+        sim_mode="$(arg sim_mode)"/>
+    <!-- Gazebo plugin: only injected when sim_mode == 'gazebo'. -->
+    <xacro:if value="${'$(arg sim_mode)' == 'gazebo'}">
+        <gazebo>
+            <plugin filename="gz_ros2_control-system" name="gz_ros2_control::GazeboSimROS2ControlPlugin">
+                <parameters>$(find abb_irb14050_gazebo)/config/controllers_gazebo.yaml</parameters>
+            </plugin>
+        </gazebo>
+    </xacro:if>
 </robot>

Commit message: feat(moveit): actualiza configuración del brazo, límites, urdf y añade launch para robot físico

File: irb14050_ws/src/abb_irb14050_moveit_config/config/abb_irb14050.ros2_control.xacro (robot description, xacro)
@@ -1,11 +1,36 @@
 <?xml version="1.0"?>
 <robot xmlns:xacro="http://www.ros.org/wiki/xacro">
-    <xacro:macro name="abb_irb14050_ros2_control" params="name initial_positions_file">
-        <xacro:property name="initial_positions" value="${xacro.load_yaml(initial_positions_file)['initial_positions']}"/>
+    <!--
+        ros2_control macro for the ABB IRB 14050.
+        Selects hardware plugin based on `sim_mode`:
+          - gazebo → gz_ros2_control/GazeboSimSystem + gz_ros2_control system plugin
+          - anything else (mock, real, etc.) → mock_components/GenericSystem
+        For the real robot, eventually replace the <xacro:unless> branch with a
+        third condition pointing to the custom EGM hardware_interface plugin.
+        Kept binary (gazebo vs everything-else) for now to avoid xacro evaluation
+        quirks observed with three-way string comparisons.
+        CRITICAL plugin name detail:
+          - The HARDWARE plugin inside <ros2_control><hardware> is named
+            `gz_ros2_control/GazeboSimSystem`
+          - The SYSTEM plugin inside <gazebo><plugin> is named
+            `gz_ros2_control::GazeboSimROS2ControlPlugin`  (NOT ...System)
+          - The library file is `gz_ros2_control-system`
+          The two are different plugins from the same .so file. Mixing them up
+          gives a "library does not contain requested plugin" error from gz_sim.
+    -->
+    <xacro:macro name="abb_irb14050_ros2_control"
+                 params="name initial_positions_file sim_mode">
+        <xacro:property name="initial_positions"
+                        value="${xacro.load_yaml(initial_positions_file)['initial_positions']}"/>
         <ros2_control name="${name}" type="system">
             <hardware>
-                <!-- By default, set up controllers for simulation. This won't work on real hardware -->
-                <plugin>mock_components/GenericSystem</plugin>
+                <xacro:if value="${sim_mode == 'gazebo'}">
+                    <plugin>gz_ros2_control/GazeboSimSystem</plugin>
+                </xacro:if>
+                <xacro:unless value="${sim_mode == 'gazebo'}">
+                    <plugin>mock_components/GenericSystem</plugin>
+                </xacro:unless>
             </hardware>
+            <!-- Arm joints (joint_1 .. joint_7) -->
             <joint name="joint_1">
                 <command_interface name="position"/>
@@ -57,5 +82,32 @@
                 <state_interface name="velocity"/>
             </joint>
+            <!-- Gripper joints (prismatic, l/r) -->
+            <joint name="gripper_joint_l">
+                <command_interface name="position"/>
+                <state_interface name="position">
+                  <param name="initial_value">${initial_positions['gripper_joint_l']}</param>
+                </state_interface>
+                <state_interface name="velocity"/>
+            </joint>
+            <joint name="gripper_joint_r">
+                <command_interface name="position"/>
+                <state_interface name="position">
+                  <param name="initial_value">${initial_positions['gripper_joint_r']}</param>
+                </state_interface>
+                <state_interface name="velocity"/>
+            </joint>
         </ros2_control>
+        <!--
+            Gazebo system plugin block — only emitted when sim_mode == 'gazebo'.
+            The `name` attribute MUST be GazeboSimROS2ControlPlugin (not System).
+        -->
+        <xacro:if value="${sim_mode == 'gazebo'}">
+            <gazebo>
+                <plugin filename="gz_ros2_control-system"
+                        name="gz_ros2_control::GazeboSimROS2ControlPlugin">
+                    <parameters>$(find abb_irb14050_gazebo)/config/controllers_gazebo.yaml</parameters>
+                </plugin>
+            </gazebo>
+        </xacro:if>
     </xacro:macro>
 </robot>

File: irb14050_ws/src/abb_irb14050_moveit_config/config/abb_irb14050.urdf.xacro (robot description, xacro)
@@ -1,9 +1,22 @@
 <?xml version="1.0"?>
 <robot xmlns:xacro="http://www.ros.org/wiki/xacro" name="abb_irb14050">
-    <xacro:arg name="initial_positions_file" default="initial_positions.yaml" />
-    <!-- Import abb_irb14050 urdf file -->
-    <xacro:include filename="$(find abb_irb14050_description)/urdf/abb_irb14050.urdf" />
-    <!-- Import control_xacro -->
-    <xacro:include filename="abb_irb14050.ros2_control.xacro" />
-    <xacro:abb_irb14050_ros2_control name="FakeSystem" initial_positions_file="$(arg initial_positions_file)"/>
+    <!--
+        Top-level xacro. Declares the public arguments and wires the
+        ros2_control macro with the chosen simulation mode.
+        sim_mode values:
+          - mock   → mock_components/GenericSystem (default; RViz-only)
+          - gazebo → gz_ros2_control/GazeboSimSystem + <gazebo><plugin> block
+          - real   → placeholder for EGM hardware_interface (currently mock)
+    -->
+    <xacro:arg name="initial_positions_file" default="initial_positions.yaml"/>
+    <xacro:arg name="sim_mode" default="mock"/>
+    <!-- Import the kinematic description (links, joints, meshes) -->
+    <xacro:include filename="$(find abb_irb14050_description)/urdf/abb_irb14050.urdf"/>
+    <!-- Import the ros2_control macro definition -->
+    <xacro:include filename="abb_irb14050.ros2_control.xacro"/>
+    <!-- Instantiate ros2_control with the runtime-selected backend -->
+    <xacro:abb_irb14050_ros2_control
+        name="IRB14050System"
+        initial_positions_file="$(arg initial_positions_file)"
+        sim_mode="$(arg sim_mode)"/>
 </robot>

Commit message: fix: restaura versión exacta de la carpeta local, sobreescribiendo el merge

File: irb14050_ws/src/abb_irb14050_moveit_config/config/abb_irb14050.ros2_control.xacro (robot description, xacro)
@@ -31,25 +31,4 @@
                     <plugin>mock_components/GenericSystem</plugin>
                 </xacro:unless>
-    <!--
-        sim_mode: selects the hardware interface plugin loaded by ros2_control.
-            - "mock"   : mock_components/GenericSystem  (no physics, RViz testing)
-            - "gazebo" : gz_ros2_control/GazeboSimSystem (Gazebo Harmonic)
-            - "real"   : (placeholder — wire EGM hardware interface here in the future)
-    -->
-    <xacro:macro name="abb_irb14050_ros2_control" params="name initial_positions_file sim_mode:=mock">
-        <xacro:property name="initial_positions" value="${xacro.load_yaml(initial_positions_file)['initial_positions']}"/>
-        <ros2_control name="${name}" type="system">
-            <hardware>
-                <xacro:if value="${sim_mode == 'mock'}">
-                    <plugin>mock_components/GenericSystem</plugin>
-                </xacro:if>
-                <xacro:if value="${sim_mode == 'gazebo'}">
-                    <plugin>gz_ros2_control/GazeboSimSystem</plugin>
-                </xacro:if>
-                <!-- Future: real robot via EGM
-                <xacro:if value="${sim_mode == 'real'}">
-                    <plugin>abb_irb14050_egm/EGMHardwareInterface</plugin>
-                </xacro:if>
-                -->
             </hardware>
             <!-- Arm joints (joint_1 .. joint_7) -->

File: irb14050_ws/src/abb_irb14050_moveit_config/config/abb_irb14050.urdf.xacro (robot description, xacro)
@@ -1,6 +1,4 @@
 <?xml version="1.0"?>
 <robot xmlns:xacro="http://www.ros.org/wiki/xacro" name="abb_irb14050">
-    <xacro:arg name="initial_positions_file" default="initial_positions.yaml" />
-    <xacro:arg name="sim_mode" default="mock" />
     <!--
         Top-level xacro. Declares the public arguments and wires the
@@ -22,15 +20,3 @@
         initial_positions_file="$(arg initial_positions_file)"
         sim_mode="$(arg sim_mode)"/>
-    <xacro:abb_irb14050_ros2_control
-        name="ABB_IRB14050_System"
-        initial_positions_file="$(arg initial_positions_file)"
-        sim_mode="$(arg sim_mode)"/>
-    <!-- Gazebo plugin: only injected when sim_mode == 'gazebo'. -->
-    <xacro:if value="${'$(arg sim_mode)' == 'gazebo'}">
-        <gazebo>
-            <plugin filename="gz_ros2_control-system" name="gz_ros2_control::GazeboSimROS2ControlPlugin">
-                <parameters>$(find abb_irb14050_gazebo)/config/controllers_gazebo.yaml</parameters>
-            </plugin>
-        </gazebo>
-    </xacro:if>
 </robot>
