Commit message: feat(description): actualiza URDF y añade meshes de gripper

File: irb14050_ws/src/abb_irb14050_description/urdf/abb_irb14050.urdf (robot description, URDF)
Before this commit: robot abb_irb14050, 10 links, 9 joints
Links:
- added link grasp_link
- added link gripper_base, mass 0.2; collision mesh filename=package://abb_irb14050_description/meshes/gripper/coarse/ba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; visual mesh filename=package://abb_irb14050_description/meshes/gripper/base.stl
- added link gripper_finger_l, mass 0.1; collision mesh filename=package://abb_irb14050_description/meshes/gripper/coarse/fi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; visual mesh filename=package://abb_irb14050_description/meshes/gripper/finger.stl
- added link gripper_finger_r, mass 0.1; collision mesh filename=package://abb_irb14050_description/meshes/gripper/coarse/fi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; visual mesh filename=package://abb_irb14050_description/meshes/gripper/finger.stl
Joints:
- added joint grasp_joint: type fixed, parent gripper_base, child grasp_link, origin xyz=0 0 0.13 rpy=0 0 0
- added joint gripper_joint_l: type prismatic, parent gripper_base, child gripper_finger_l, origin xyz=0 0.0065 0.0837 rpy=0 0 3.14159265359, axis -1 0 0, limit lower=-0.001 upper=0.025 effort=20 velocity=2
- added joint gripper_joint_r: type prismatic, parent gripper_base, child gripper_finger_r, origin xyz=0 -0.0065 0.0837 rpy=0 0 0, axis -1 0 0, limit lower=-0.001 upper=0.025 effort=20 velocity=2
- added joint gripper_mount_joint: type fixed, parent tool0, child gripper_base, origin xyz=0 0 0 rpy=0 0 0
